Commit message: 更新gazebo仿真插件的配置

File: learning_gazebo/urdf/sensors/camera_gazebo.xacro (robot description, xacro)
@@ -49,16 +49,12 @@
                 </camera>
                 <plugin name="gazebo_camera" filename="libgazebo_ros_camera.so">
-                    <alwaysOn>true</alwaysOn>
-                    <updateRate>0.0</updateRate>
-                    <cameraName>/camera</cameraName>
-                    <imageTopicName>image_raw</imageTopicName>
-                    <cameraInfoTopicName>camera_info</cameraInfoTopicName>
-                    <frameName>camera_link</frameName>
-                    <hackBaseline>0.07</hackBaseline>
-                    <distortionK1>0.0</distortionK1>
-                    <distortionK2>0.0</distortionK2>
-                    <distortionK3>0.0</distortionK3>
-                    <distortionT1>0.0</distortionT1>
-                    <distortionT2>0.0</distortionT2>
+				    <ros>
+				        <!-- <namespace>stereo</namespace> -->
+				        <remapping>~/image_raw:=image_raw</remapping>
+				        <remapping>~/camera_info:=camera_info</remapping>
+				    </ros>
+				    <camera_name>${prefix}</camera_name>
+				    <frame_name>${prefix}_link</frame_name>
+				    <hack_baseline>0.2</hack_baseline>
                 </plugin>
             </sensor>

File: learning_gazebo/urdf/sensors/kinect_gazebo.xacro (robot description, xacro)
@@ -9,5 +9,5 @@
                 <origin xyz="0 0 0" rpy="0 0 ${M_PI/2}"/>
                 <geometry>
-                    <mesh filename="package://mbot_description/meshes/kinect.dae" />
+                    <mesh filename="package://learning_gazebo/meshes/kinect.dae" />
                 </geometry>
             </visual>
@@ -27,6 +27,7 @@
             <sensor type="depth" name="${prefix}">
                 <always_on>true</always_on>
-                <update_rate>20.0</update_rate>
-                <camera>
+                <update_rate>15.0</update_rate>
+                <pose>0 0 0 0 0 0</pose>
+                <camera name="kinect">
                     <horizontal_fov>${60.0*M_PI/180.0}</horizontal_fov>
                     <image>
@@ -40,21 +41,18 @@
                     </clip>
                 </camera>
-                <plugin name="kinect_${prefix}_controller" filename="libgazebo_ros_openni_kinect.so">
-                    <cameraName>${prefix}</cameraName>
-                    <alwaysOn>true</alwaysOn>
-                    <updateRate>10</updateRate>
-                    <imageTopicName>rgb/image_raw</imageTopicName>
-                    <depthImageTopicName>depth/image_raw</depthImageTopicName>
-                    <pointCloudTopicName>depth/points</pointCloudTopicName>
-                    <cameraInfoTopicName>rgb/camera_info</cameraInfoTopicName>
-                    <depthImageCameraInfoTopicName>depth/camera_info</depthImageCameraInfoTopicName>
-                    <frameName>${prefix}_frame_optical</frameName>
-                    <baseline>0.1</baseline>
-                    <distortion_k1>0.0</distortion_k1>
-                    <distortion_k2>0.0</distortion_k2>
-                    <distortion_k3>0.0</distortion_k3>
-                    <distortion_t1>0.0</distortion_t1>
-                    <distortion_t2>0.0</distortion_t2>
-                    <pointCloudCutoff>0.4</pointCloudCutoff>
+                <plugin name="${prefix}_controller" filename="libgazebo_ros_camera.so">
+		 		 	<ros>
+						<!-- <namespace>${prefix}</namespace> -->
+						<remapping>${prefix}/image_raw:=rgb/image_raw</remapping>
+						<remapping>${prefix}/image_depth:=depth/image_raw</remapping>
+						<remapping>${prefix}/camera_info:=rgb/camera_info</remapping>
+						<remapping>${prefix}/camera_info_depth:=depth/camera_info</remapping>
+						<remapping>${prefix}/points:=depth/points</remapping>
+					</ros>
+					<camera_name>${prefix}</camera_name>
+					<frame_name>${prefix}_frame_optical</frame_name>
+				    <hack_baseline>0.07</hack_baseline>
+				    <min_depth>0.001</min_depth>
+				    <max_depth>300.0</max_depth>
                 </plugin>
             </sensor>

File: learning_gazebo/urdf/sensors/lidar_gazebo.xacro (robot description, xacro)
@@ -30,7 +30,5 @@
         <gazebo reference="${prefix}_link">
             <sensor type="ray" name="rplidar">
-                <pose>0 0 0 0 0 0</pose>
-                <visualize>false</visualize>
-                <update_rate>5.5</update_rate>
+                <update_rate>20</update_rate>
                 <ray>
                     <scan>
@@ -44,5 +42,5 @@
                     <range>
                       <min>0.10</min>
-                      <max>6.0</max>
+                      <max>30.0</max>
                       <resolution>0.01</resolution>
                     </range>
@@ -53,7 +51,10 @@
                     </noise>
                 </ray>
-                <plugin name="gazebo_rplidar" filename="libgazebo_ros_laser.so">
-                    <topicName>/scan</topicName>
-                    <frameName>laser_link</frameName>
+                <plugin name="gazebo_rplidar" filename="libgazebo_ros_ray_sensor.so">
+		      <ros>
+			<namespace>/</namespace>
+			<remapping>~/out:=scan</remapping>
+		      </ros>
+		      <output_type>sensor_msgs/LaserScan</output_type>
                 </plugin>
             </sensor>

File: learning_urdf/urdf/sensors/kinect_gazebo.xacro (robot description, xacro)
@@ -9,5 +9,5 @@
                 <origin xyz="0 0 0" rpy="0 0 ${M_PI/2}"/>
                 <geometry>
-                    <mesh filename="package://mbot_description/meshes/kinect.dae" />
+                    <mesh filename="package://learning_urdf/meshes/kinect.dae" />
                 </geometry>
             </visual>
@@ -27,6 +27,7 @@
             <sensor type="depth" name="${prefix}">
                 <always_on>true</always_on>
-                <update_rate>20.0</update_rate>
-                <camera>
+                <update_rate>15.0</update_rate>
+                <pose>0 0 0 0 0 0</pose>
+                <camera name="kinect">
                     <horizontal_fov>${60.0*M_PI/180.0}</horizontal_fov>
                     <image>
@@ -40,21 +41,18 @@
                     </clip>
                 </camera>
-                <plugin name="kinect_${prefix}_controller" filename="libgazebo_ros_openni_kinect.so">
-                    <cameraName>${prefix}</cameraName>
-                    <alwaysOn>true</alwaysOn>
-                    <updateRate>10</updateRate>
-                    <imageTopicName>rgb/image_raw</imageTopicName>
-                    <depthImageTopicName>depth/image_raw</depthImageTopicName>
-                    <pointCloudTopicName>depth/points</pointCloudTopicName>
-                    <cameraInfoTopicName>rgb/camera_info</cameraInfoTopicName>
-                    <depthImageCameraInfoTopicName>depth/camera_info</depthImageCameraInfoTopicName>
-                    <frameName>${prefix}_frame_optical</frameName>
-                    <baseline>0.1</baseline>
-                    <distortion_k1>0.0</distortion_k1>
-                    <distortion_k2>0.0</distortion_k2>
-                    <distortion_k3>0.0</distortion_k3>
-                    <distortion_t1>0.0</distortion_t1>
-                    <distortion_t2>0.0</distortion_t2>
-                    <pointCloudCutoff>0.4</pointCloudCutoff>
+                <plugin name="kinect_${prefix}_controller" filename="libgazebo_ros_camera.so">
+		 		 	<ros>
+						<!-- <namespace>${prefix}</namespace> -->
+						<remapping>${prefix}/image_raw:=rgb/image_raw</remapping>
+						<remapping>${prefix}/image_depth:=depth/image_raw</remapping>
+						<remapping>${prefix}/camera_info:=rgb/camera_info</remapping>
+						<remapping>${prefix}/camera_info_depth:=depth/camera_info</remapping>
+						<remapping>${prefix}/points:=depth/points</remapping>
+					</ros>
+					<camera_name>${prefix}</camera_name>
+					<frame_name>${prefix}_frame_optical</frame_name>
+				    <hack_baseline>0.07</hack_baseline>
+				    <min_depth>0.001</min_depth>
+				    <max_depth>300.0</max_depth>
                 </plugin>
             </sensor>
