Commit message: 修复gazebo仿真的bug

File: learning_gazebo/urdf/sensors/kinect_gazebo.xacro (robot description, xacro)
@@ -9,5 +9,5 @@
                 <origin xyz="0 0 0" rpy="0 0 ${M_PI/2}"/>
                 <geometry>
-                    <mesh filename="package://learning_gazebo/meshes/kinect.dae" />
+                    <box size="0.15 0.04 0.04" />
                 </geometry>
             </visual>
